File: pcbs/main.kicad_pcb (KiCad board)
At the start: 2 copper layers, 261.1 x 103.7 mm, 91 parts

Commit message: added two more mounting holes
Parts:
- added REF**: TestPoint_Plated_Hole_D2.0mm, TestPoint:TestPoint_Plated_Hole_D2.0mm, F.Cu at (108.8, 142.2)
- added REF**: TestPoint_Plated_Hole_D2.0mm, TestPoint:TestPoint_Plated_Hole_D2.0mm, F.Cu at (248.0, 142.6)

Commit message: a few more mounting holes to make sure the case is attached well
Parts:
- added REF**: TestPoint_Plated_Hole_D2.0mm, TestPoint:TestPoint_Plated_Hole_D2.0mm, F.Cu at (92.2, 137.2)
- added REF**: TestPoint_Plated_Hole_D2.0mm, TestPoint:TestPoint_Plated_Hole_D2.0mm, F.Cu at (201.9, 152.7)
- added REF**: TestPoint_Plated_Hole_D2.0mm, TestPoint:TestPoint_Plated_Hole_D2.0mm, F.Cu at (265.6, 137.2)
- added REF**: TestPoint_Plated_Hole_D2.0mm, TestPoint:TestPoint_Plated_Hole_D2.0mm, F.Cu at (219.6, 91.1)
- added REF**: TestPoint_Plated_Hole_D2.0mm, TestPoint:TestPoint_Plated_Hole_D2.0mm, F.Cu at (155.9, 152.7)
