File: pcbs/main.kicad_pcb (KiCad board)
At the start: 2 copper layers, 261.1 x 103.7 mm, 98 parts

Commit message: minor changes to the routing
Routing:
- net P9: track 330.9 -> 332.1 mm
- net P8: track 303.6 -> 304.6 mm
- net P7: track 328.3 -> 329.2 mm
- net P6: track 293.3 -> 294.1 mm
- net P5: track 348.5 -> 349.1 mm
- net P4: track 386.5 -> 387.1 mm
- added copper zone on B.Cu, net (none)
- added copper zone on F.Cu, net (none)
